Commit message: update the object urdf
1. Define the initial rotation in urdf file instead of the start rotation defined in InHandManipulation.py
2. Update object property in urdf file
3. Add object "cross"
4. Update .gitignore

File: environments/InHandManipulation/definitions/additional_urdfs/rect.urdf (robot description, URDF)
Before this commit: robot rect, 1 links, 0 joints
Links:
- link rect: geometry collision box size=0.25 2.5 1; visual box size=0.25 2.5 1
