Commit message: update physical and collision properties of the objects

File: environments/InHandManipulation/definitions/additional_urdfs/ball.urdf (robot description, URDF)
Before this commit: robot box, 1 links, 0 joints
Links:
- removed link box
- added link ball, mass 0.01; collision sphere radius=0.5; visual sphere radius=0.5

File: environments/InHandManipulation/definitions/additional_urdfs/bunny.urdf (robot description, URDF)
Before this commit: robot cube.urdf, 1 links, 0 joints
Links:
- link baseLink: mass 0.01 -> 0.0001

File: environments/InHandManipulation/definitions/additional_urdfs/duck.urdf (robot description, URDF)
Before this commit: robot cube.urdf, 1 links, 0 joints
Links:
- link baseLink: mass .01 -> .0001

File: environments/InHandManipulation/definitions/additional_urdfs/teddy.urdf (robot description, URDF)
Before this commit: robot cube.urdf, 1 links, 0 joints
Links:
- link baseLink: mass .01 -> 0.01
